File: GTB.kicad_pcb (KiCad board)
At the start: 2 copper layers, 7 parts

Commit message: Completed Tutorial
Parts:
- BT1: moved to B.Cu
- moved R2 229.9 mm to (204.5, 77.5), turned to 270 degrees
- moved TU1 225.8 mm to (212.1, 71.1), turned to 270 degrees
- moved R1 224.9 mm to (218.4, 71.1), turned to 270 degrees
- moved VR1 218.3 mm to (220.5, 62.5), turned to 180 degrees
- moved D1 213.7 mm to (210.8, 80.0)
- moved C1 198.4 mm to (204.5, 66.0), turned to 90 degrees
- moved BT1 198.1 mm to (212.1, 71.1), turned to 180 degrees
Routing:
- net GND: track 0.00 -> 18.3 mm, vias 0 -> 2
- net N-000001: track 0.00 -> 17.3 mm
- net N-000006: track 0.00 -> 10.9 mm
- net N-000002: track 0.00 -> 8.14 mm
- net N-000003: track 0.00 -> 5.30 mm
- added copper zone on B.Cu, net GND
- added copper zone on F.Cu, net VCC
Other:
- board outline added: 25.4 x 25.4 mm
